File: Capacitor-Tester_v0_0_1/capacitor-tester_v0.0.1.brd (EAGLE design)
At the start: 100 x 80 mm, 38 parts, among them IC1 AD8531ARZ, IC2 MC34063EBD-TR, IC3 DAC6571IDBVT, IC4 AD8531ARZ, J1 USB4125-GF-A-0190_REVA2, J2 DS1044-140G, J4 250-103, U1 AD5933, U2 LM6171AIMX/NOPB, Y1 LFSPXO018034

Commit message: v0.0.1 - Version control before big changes in the schematic
Parts:
- removed C3, C7: 1u, custom_library:C0603
- removed R15, R16, R5, R6: 20k-1%, custom_library:R0603
- R13: value 20k-1% -> 5k-1%
- R14: value 4k-1% -> 10k-1%
- R2: value 20k-1% -> 10k-1%
- R4: value 4k-1% -> 1k-1%
Connections:
- removed net N$12: C7.1, IC4.3, R15.2, R16.1
- removed net N$4: C3.1, IC1.3, R5.2, R6.1
- removed net OPAMP_OUT: IC1.6, IC4.6, J2.1, J2.2, J2.3, J2.4, J2.5, J2.6, J2.7, R14.2, R4.2
- new net UZA_OUT: IC1.6, J2.1, J2.2, J2.3, J2.4, J2.5, J2.6, J2.7, R4.2
- new net UZB_OUT: IC1.3, IC4.6, R14.2
- net +5V: no longer R15.1, R5.1
- net DAC_OUT: now also IC4.3
- net GND: now also R13.2; no longer C3.2, C7.2, R16.2, R6.2
- net VOUT: no longer R13.2
Changed lines of the file:
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@@
 <attribute name="VALUE" x="-2.712" y="-108.31" size="1.27" layer="27" align="center"/>
 </element>
-<element name="R2" library="custom_library" package="R0603" value="20k-1%" x="-15" y="-111.2" smashed="yes">
+<element name="R2" library="custom_library" package="R0603" value="10k-1%" x="-15" y="-111.2" smashed="yes">
 <attribute name="NAME" x="-16.32476875" y="-110.213721875" size="0.52744375" layer="25"/>
 <attribute name="VALUE" x="-16.719259375" y="-112.72958125" size="0.525771875" layer="27"/>
 </element>
-<element name="R4" library="custom_library" package="R0603" value="4k-1%" x="-18.4" y="-111.2" smashed="yes">
+<element name="R4" library="custom_library" package="R0603" value="1k-1%" x="-18.4" y="-111.2" smashed="yes">
 <attribute name="NAME" x="-19.72476875" y="-110.213721875" size="0.52744375" layer="25"/>
 <attribute name="VALUE" x="-20.119259375" y="-112.72958125" size="0.525771875" layer="27"/>
-</element>
-<element name="C3" library="custom_library" package="C0603" value="1u" x="-17.8" y="-115.2" smashed="yes">
-<attribute name="NAME" x="-19.635" y="-114.565" size="0.8" layer="25"/>
-<attribute name="VALUE" x="-18.435" y="-117.105" size="1.27" layer="27"/>
-</element>
-<element name="R5" library="custom_library" package="R0603" value="20k-1%" x="-21.8" y="-115.4" smashed="yes">
-<attribute name="NAME" x="-23.12476875" y="-114.413721875" size="0.52744375" layer="25"/>
-<attribute name="VALUE" x="-23.519259375" y="-116.92958125" size="0.525771875" layer="27"/>
-</element>
-<element name="R6" library="custom_library" package="R0603" value="20k-1%" x="-25.2" y="-115.4" smashed="yes">
-<attribute name="NAME" x="-26.52476875" y="-114.413721875" size="0.52744375" layer="25"/>
-<attribute name="VALUE" x="-26.919259375" y="-116.92958125" size="0.525771875" layer="27"/>
 </element>
 <element name="J2" library="DS1044-140G" package="CONNFLY_DS1044-140G" value="DS1044-140G" x="-3.81" y="-135.72" smashed="yes">
@@
 <attribute name="NAME" x="-107.6" y="-221.39" size="1.27" layer="25" align="center"/>
 </element>
-<element name="R13" library="custom_library" package="R0603" value="20k-1%" x="-104.6" y="-229.6" smashed="yes">
+<element name="R13" library="custom_library" package="R0603" value="5k-1%" x="-104.6" y="-229.6" smashed="yes">
 <attribute name="NAME" x="-105.92476875" y="-228.613721875" size="0.52744375" layer="25"/>
 <attribute name="VALUE" x="-106.319259375" y="-231.12958125" size="0.525771875" layer="27"/>
 </element>
-<element name="R14" library="custom_library" package="R0603" value="4k-1%" x="-109" y="-233.8" smashed="yes">
+<element name="R14" library="custom_library" package="R0603" value="10k-1%" x="-109" y="-233.8" smashed="yes">
 <attribute name="NAME" x="-110.32476875" y="-232.813721875" size="0.52744375" layer="25"/>
 <attribute name="VALUE" x="-110.719259375" y="-235.32958125" size="0.525771875" layer="27"/>
-</element>
-<element name="C7" library="custom_library" package="C0603" value="1u" x="-108.8" y="-229.6" smashed="yes">
-<attribute name="NAME" x="-110.635" y="-228.965" size="0.8" layer="25"/>
-<attribute name="VALUE" x="-109.435" y="-231.505" size="1.27" layer="27"/>
-</element>
-<element name="R15" library="custom_library" package="R0603" value="20k-1%" x="-105.4" y="-233.8" smashed="yes">
-<attribute name="NAME" x="-106.72476875" y="-232.813721875" size="0.52744375" layer="25"/>
-<attribute name="VALUE" x="-107.119259375" y="-235.32958125" size="0.525771875" layer="27"/>
-</element>
-<element name="R16" library="custom_library" package="R0603" value="20k-1%" x="-101.8" y="-233.8" smashed="yes">
-<attribute name="NAME" x="-103.12476875" y="-232.813721875" size="0.52744375" layer="25"/>
-<attribute name="VALUE" x="-103.519259375" y="-235.32958125" size="0.525771875" layer="27"/>
 </element>
 <element name="C8" library="custom_library" package="C0603" value="10u" x="-108.8" y="-237.8" smashed="yes">
@@
 <contactref element="J1" pad="S3"/>
 <contactref element="IC1" pad="4"/>
-<contactref element="C3" pad="2"/>
-<contactref element="R6" pad="2"/>
 <contactref element="U2" pad="4"/>
 <contactref element="U2" pad="3"/>
@@
 <contactref element="IC3" pad="6"/>
 <contactref element="IC4" pad="4"/>
-<contactref element="C7" pad="2"/>
-<contactref element="R16" pad="2"/>
 <contactref element="C8" pad="2"/>
+<contactref element="R13" pad="2"/>
 <wire x1="-44.61" y1="-181.6" x2="-51.5" y2="-188" width="0" layer="19" extent="1-1"/>
 <wire x1="-39.3" y1="-188" x2="-44.61" y2="-181.6" width="0" layer="19" extent="1-1"/>
@@
 <wire x1="-105.45" y1="-215.8" x2="-102.95" y2="-214.85" width="0" layer="19" extent="1-1"/>
 <wire x1="-110.312" y1="-227.105" x2="-105.45" y2="-215.8" width="0" layer="19" extent="1-1"/>
-<wire x1="-107.95" y1="-229.6" x2="-110.312" y2="-227.105" width="0" layer="19" extent="1-1"/>
-<wire x1="-101.01" y1="-233.8" x2="-107.95" y2="-229.6" width="0" layer="19" extent="1-1"/>
-<wire x1="-107.95" y1="-237.8" x2="-101.01" y2="-233.8" width="0" layer="19" extent="1-1"/>
-<wire x1="-16.95" y1="-115.2" x2="-4.94" y2="-165.84" width="0" layer="19" extent="1-1"/>
-<wire x1="-24.41" y1="-115.4" x2="-16.95" y2="-115.2" width="0" layer="19" extent="1-1"/>
-<wire x1="-5.424" y1="-110.215" x2="-16.95" y2="-115.2" width="0" layer="19" extent="1-1"/>
+<wire x1="-103.81" y1="-229.6" x2="-110.312" y2="-227.105" width="0" layer="19" extent="1-1"/>
+<wire x1="-107.95" y1="-237.8" x2="-103.81" y2="-229.6" width="0" layer="19" extent="1-1"/>
+<wire x1="-5.424" y1="-110.215" x2="-4.94" y2="-165.84" width="0" layer="19" extent="1-1"/>
 <wire x1="-8.92" y1="-82.2" x2="-5.424" y2="-110.215" width="0" layer="19" extent="1-1"/>
 <wire x1="-8.92" y1="-78.4" x2="-8.92" y2="-82.2" width="0" layer="19" extent="1-1"/>
@@
 <contactref element="R1" pad="2"/>
 <contactref element="IC1" pad="7"/>
-<contactref element="R5" pad="1"/>
 <contactref element="IC2" pad="6"/>
 <contactref element="C5" pad="1"/>
@@
 <contactref element="IC3" pad="3"/>
 <contactref element="IC4" pad="7"/>
-<contactref element="R15" pad="1"/>
 <contactref element="C8" pad="1"/>
 <wire x1="-56.5" y1="-188" x2="-61.19" y2="-189.2" width="0" layer="19" extent="1-1"/>
@@
 <wire x1="-105.45" y1="-216.75" x2="-61.19" y2="-189.2" width="0" layer="19" extent="1-1"/>
 <wire x1="-104.888" y1="-224.565" x2="-105.45" y2="-216.75" width="0" layer="19" extent="1-1"/>
-<wire x1="-106.19" y1="-233.8" x2="-104.888" y2="-224.565" width="0" layer="19" extent="1-1"/>
-<wire x1="-109.65" y1="-237.8" x2="-106.19" y2="-233.8" width="0" layer="19" extent="1-1"/>
-<wire x1="-22.59" y1="-115.4" x2="-28.288" y2="-173.235" width="0" layer="19" extent="1-1"/>
-<wire x1="0" y1="-107.675" x2="-22.59" y2="-115.4" width="0" layer="19" extent="1-1"/>
+<wire x1="-109.65" y1="-237.8" x2="-104.888" y2="-224.565" width="0" layer="19" extent="1-1"/>
+<wire x1="0" y1="-107.675" x2="-28.288" y2="-173.235" width="0" layer="19" extent="1-1"/>
 <wire x1="-6.41" y1="-86.8" x2="0" y2="-107.675" width="0" layer="19" extent="1-1"/>
 <wire x1="-10.41" y1="-86.8" x2="-6.41" y2="-86.8" width="0" layer="19" extent="1-1"/>
@@
 <contactref element="U1" pad="6"/>
 <contactref element="R2" pad="2"/>
-<contactref element="R13" pad="2"/>
 <wire x1="-7.01" y1="-15.95" x2="-14.21" y2="-111.2" width="0" layer="19" extent="1-1"/>
-<wire x1="-103.81" y1="-229.6" x2="-14.21" y2="-111.2" width="0" layer="19" extent="1-1"/>
 </signal>
 <signal name="N$1">
@@
 <wire x1="-5.424" y1="-107.675" x2="-15.79" y2="-111.2" width="0" layer="19" extent="1-1"/>
 </signal>
-<signal name="OPAMP_OUT">
+<signal name="UZA_OUT">
 <contactref element="IC1" pad="6"/>
 <contactref element="R4" pad="2"/>
@@
 <contactref element="J2" pad="3"/>
 <contactref element="J2" pad="2"/>
-<contactref element="IC4" pad="6"/>
-<contactref element="R14" pad="2"/>
 <wire x1="-7.62" y1="-140.8" x2="-7.62" y2="-143.34" width="0" layer="19" extent="1-1"/>
 <wire x1="-7.62" y1="-138.26" x2="-7.62" y2="-140.8" width="0" layer="19" extent="1-1"/>
@@
 <wire x1="-17.61" y1="-111.2" x2="-7.62" y2="-128.1" width="0" layer="19" extent="1-1"/>
 <wire x1="0" y1="-108.945" x2="-17.61" y2="-111.2" width="0" layer="19" extent="1-1"/>
-<wire x1="-104.888" y1="-225.835" x2="-7.62" y2="-143.34" width="0" layer="19" extent="1-1"/>
-<wire x1="-108.21" y1="-233.8" x2="-104.888" y2="-225.835" width="0" layer="19" extent="1-1"/>
-</signal>
-<signal name="N$4">
-<contactref element="IC1" pad="3"/>
-<contactref element="C3" pad="1"/>
-<contactref element="R5" pad="2"/>
-<contactref element="R6" pad="1"/>
-<wire x1="-21.01" y1="-115.4" x2="-25.99" y2="-115.4" width="0" layer="19" extent="1-1"/>
-<wire x1="-18.65" y1="-115.2" x2="-21.01" y2="-115.4" width="0" layer="19" extent="1-1"/>
-<wire x1="-5.424" y1="-108.945" x2="-18.65" y2="-115.2" width="0" layer="19" extent="1-1"/>
 </signal>
 <signal name="N$2">
@@
 <signal name="DAC_OUT">
 <contactref element="IC3" pad="1"/>
+<contactref element="IC4" pad="3"/>
+<wire x1="-105.45" y1="-214.85" x2="-110.312" y2="-225.835" width="0" layer="19" extent="1-1"/>
 </signal>
 <signal name="N$9">
@@
 <wire x1="-110.312" y1="-224.565" x2="-105.39" y2="-229.6" width="0" layer="19" extent="1-1"/>
 </signal>
-<signal name="N$12">
-<contactref element="IC4" pad="3"/>
-<contactref element="C7" pad="1"/>
-<contactref element="R15" pad="2"/>
-<contactref element="R16" pad="1"/>
-<wire x1="-110.312" y1="-225.835" x2="-109.65" y2="-229.6" width="0" layer="19" extent="1-1"/>
-<wire x1="-104.61" y1="-233.8" x2="-109.65" y2="-229.6" width="0" layer="19" extent="1-1"/>
-<wire x1="-102.59" y1="-233.8" x2="-104.61" y2="-233.8" width="0" layer="19" extent="1-1"/>
+<signal name="UZB_OUT">
+<contactref element="R14" pad="2"/>
+<contactref element="IC4" pad="6"/>
+<contactref element="IC1" pad="3"/>
+<wire x1="-104.888" y1="-225.835" x2="-5.424" y2="-108.945" width="0" layer="19" extent="1-1"/>
+<wire x1="-108.21" y1="-233.8" x2="-104.888" y2="-225.835" width="0" layer="19" extent="1-1"/>
 </signal>
 </signals>
